File: HTMDv2.1.kicad_pcb (KiCad board)
At the start: 4 copper layers, 90 x 55 mm, 118 parts, among them IC1 TJA1441AT_0Z, J1 Conn_02x20_Odd_Even, J2 Conn_02x20_Odd_Even, J3 MothreCANConn, J4 XT60PW-F, J5 XT60PW-F, J6 Conn_01x06, SW1 SW_Push, SW2 SW_Push, U1 ADP3338AKCZ-3.3, U10 TC74LCXC00FT, U11 TC7S14FU, U12 ADuM7223, U13 SQJ180EP-T1_GE3, U14 SQJ180EP-T1_GE3, U15 SQJ180EP-T1_GE3, U16 SQJ180EP-T1_GE3, U17 ADuM7223, U18 ADuM7223, U19 SQJ180EP-T1_GE3, U2 NJM78L12SU3, U20 SQJ180EP-T1_GE3, U21 SQJ180EP-T1_GE3, U22 SQJ180EP-T1_GE3, U23 ADuM7223, U3 TC74LCXC00FT, U4 TC7S32FU, U5 TC74LCXC00FT, U6 TC7S14FU, U7 ESP32-PICO-D4_EXP, U8 TC74LCXC00FT, U9 TC7S32FU

Commit message: Artwork finish
Parts:
- removed C28, C33, C34, C39, C5: 0.1u, Capacitor_SMD:C_0402_1005Metric
- removed C29, C30, C31, C32, C35, C36, C37, C38, C6: 10u, Capacitor_SMD:C_0805_2012Metric
- removed C4: 1u, Capacitor_SMD:C_0402_1005Metric
- removed D10, D11, D12, D13: SS2040FL, 0-Myparts:SS2040FL
- removed D2, D3, D4, D5, D9: BAT43XV2, 0-Myparts:BAT43XV2
- removed U10, U8: TC74LCXC00FT, 0-Myparts:TC74AC00FTEL
- removed U11, U6: TC7S14FU, 0-Myparts:TC7S14FU
- removed U12, U17, U18, U23: ADuM7223, 0-Myparts:ADuM7223
- removed U2: NJM78L12SU3, 0-Myparts:REG_MCP1700T-3602E_MB
- removed U4, U9: TC7S32FU, 0-Myparts:TC7S32FU
- added IC2: A3921KLPTR-T, 0-Myparts:A3944KLPTRT, F.Cu at (102.4, 66.2)
- added IC3: A3921KLPTR-T, 0-Myparts:A3944KLPTRT, F.Cu at (102.4, 51.5)
- added R34: R, Resistor_SMD:R_0603_1608Metric_Pad0.98x0.95mm_HandSolder, F.Cu at (137.7, 60.6)
- added SW3: SW_Push, 0-Myparts:SKRPABE010, F.Cu at (124.6, 72.2)
- added State1.1: LED, LED_SMD:LED_0603_1608Metric_Pad1.05x0.95mm_HandSolder, F.Cu at (97.0, 58.9)
- added State1.2: LED, LED_SMD:LED_0603_1608Metric_Pad1.05x0.95mm_HandSolder, F.Cu at (100.5, 58.9)
- added State2.1: LED, LED_SMD:LED_0603_1608Metric_Pad1.05x0.95mm_HandSolder, F.Cu at (101.1, 42.9)
- added State2.2: LED, LED_SMD:LED_0603_1608Metric_Pad1.05x0.95mm_HandSolder, F.Cu at (101.1, 44.6)
- C10: value 220p -> 0.1u; footprint Capacitor_SMD:C_0402_1005Metric -> Capacitor_SMD:C_0402_1005Metric_Pad0.74x0.62mm_HandSolder; moved to B.Cu
- C11, C26: value 220p -> 10u; footprint Capacitor_SMD:C_0402_1005Metric -> Capacitor_SMD:C_0805_2012Metric_Pad1.18x1.45mm_HandSolder; moved to B.Cu
- C12, C23, C25: value 220p -> 0.1u; footprint Capacitor_SMD:C_0402_1005Metric -> Capacitor_SMD:C_0402_1005Metric_Pad0.74x0.62mm_HandSolder
- C13, C24: value 220p -> 10u; footprint Capacitor_SMD:C_0402_1005Metric -> Capacitor_SMD:C_0805_2012Metric_Pad1.18x1.45mm_HandSolder
- C14, C8: value 0.1u -> 10u; footprint Capacitor_SMD:C_0402_1005Metric -> Capacitor_SMD:C_0805_2012Metric_Pad1.18x1.45mm_HandSolder; moved to B.Cu
- C20, C27: footprint Capacitor_SMD:C_0402_1005Metric -> Capacitor_SMD:C_0402_1005Metric_Pad0.74x0.62mm_HandSolder; moved to B.Cu
- C21, C22, C7, C9: value 0.1u -> 10u; footprint Capacitor_SMD:C_0402_1005Metric -> Capacitor_SMD:C_0805_2012Metric_Pad1.18x1.45mm_HandSolder
- D6, D7, D8: value BAT43XV2 -> LED; footprint 0-Myparts:BAT43XV2 -> LED_SMD:LED_0603_1608Metric_Pad1.05x0.95mm_HandSolder
- R1: footprint Resistor_SMD:R_0603_1608Metric -> Resistor_SMD:R_0603_1608Metric_Pad0.98x0.95mm_HandSolder; moved to B.Cu
- R11: value 20k -> 1k; footprint Resistor_SMD:R_0603_1608Metric -> Resistor_SMD:R_0603_1608Metric_Pad0.98x0.95mm_HandSolder
- R12, R13, R2, R3: footprint Resistor_SMD:R_0603_1608Metric -> Resistor_SMD:R_0603_1608Metric_Pad0.98x0.95mm_HandSolder
- R14, R15, R4: value 1.8k -> 20k; footprint Resistor_SMD:R_0603_1608Metric -> Resistor_SMD:R_0603_1608Metric_Pad0.98x0.95mm_HandSolder
- R16, R17: value 1.8k -> R; footprint Resistor_SMD:R_0603_1608Metric -> Resistor_SMD:R_0603_1608Metric_Pad0.98x0.95mm_HandSolder
- R5, R7: value 1.8k -> 10k; footprint Resistor_SMD:R_0603_1608Metric -> Resistor_SMD:R_0603_1608Metric_Pad0.98x0.95mm_HandSolder
- R6: value 1.8k -> 1k; footprint Resistor_SMD:R_0603_1608Metric -> Resistor_SMD:R_0603_1608Metric_Pad0.98x0.95mm_HandSolder
- U3, U5: value TC74LCXC00FT -> ADUM140E0BRWZ-RL; footprint 0-Myparts:TC74AC00FTEL -> 0-Myparts:ADuM140ER
- U7: value ESP32-PICO-D4_EXP -> ESP32-PICO-D4
- moved R2 35.0 mm to (104.5, 42.9)
- moved R13 32.7 mm to (94.2, 58.3), turned to -90 degrees
- moved R3 32.6 mm to (104.5, 44.6)
- moved C27 31.9 mm to (93.7, 67.2), turned to -90 degrees
- moved D6 29.9 mm to (141.2, 66.4), turned to 180 degrees
- moved D7 29.8 mm to (141.1, 63.5), turned to 180 degrees
- moved C23 28.2 mm to (96.5, 70.4), turned to -90 degrees
- moved C22 27.7 mm to (94.9, 63.5)
- moved R6 27.6 mm to (110.9, 44.7), turned to 0 degrees
- moved C12 27.3 mm to (96.0, 56.5), turned to -90 degrees
- moved C7 26.4 mm to (94.2, 47.9), turned to -90 degrees
- moved C26 26.4 mm to (95.8, 67.6), turned to -90 degrees
- moved D8 26.0 mm to (141.1, 60.6), turned to 180 degrees
- moved C25 25.7 mm to (93.3, 51.9), turned to -90 degrees
- moved R1 25.5 mm to (103.5, 66.2), turned to 90 degrees
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Connections:
- C10 pad 1: GND -> +5V
- C10 pad 2: Net-(D2-K) -> GNDPWR
- C11 pad 1: GND -> +5V
- C11 pad 2: Net-(D3-K) -> GNDPWR
- C12 pad 1: GND -> +24V
- C12 pad 2: Net-(D4-K) -> GNDPWR
- C13 pad 1: GND -> Net-(IC2-CP1)
- C13 pad 2: Net-(D5-K) -> CP1
- C14 pad 1: +3.3V -> +5VA
- C14 pad 2: GND -> GNDPWR
- C20 pad 1: +3.3V -> +5VA
- C20 pad 2: GND -> GNDPWR
- C21 pad 1: +3.3V -> SA1
- C21 pad 2: GND -> Net-(IC2-SA)
- C22 pad 1: +3.3V -> SB1
- C22 pad 2: GND -> Net-(IC2-CB)
- C23 pad 1: GND -> +24V
- C23 pad 2: Net-(D6-K) -> GNDPWR
- C24 pad 1: GND -> Net-(IC3-VREG)
- C24 pad 2: Net-(D7-K) -> GNDPWR
- C25 pad 1: GND -> Net-(IC3-VREG)
- C25 pad 2: Net-(D8-K) -> GNDPWR
- C26 pad 1: GND -> Net-(IC2-VREG)
- C26 pad 2: Net-(D9-K) -> GNDPWR
- C27 pad 1: +3.3V -> Net-(IC2-VREG)
- C27 pad 2: GND -> GNDPWR
- C7 pad 1: +3.3V -> SB2
- C7 pad 2: GND -> Net-(IC3-CB)
- C8 pad 1: +3.3V -> SA2
- C8 pad 2: GND -> Net-(IC3-SA)
- C9 pad 1: +3.3V -> Net-(IC3-CP1)
- C9 pad 2: GND -> CP2
- D6 pad 1: Net-(D6-K) -> GND
- D7 pad 1: Net-(D7-K) -> GND
- D8 pad 1: Net-(D8-K) -> GND
- J4 pad 1: Net-(U17-GNDA) -> SB1
- J4 pad 2: Net-(U12-GNDA) -> SA1
- J5 pad 1: Net-(U23-GNDA) -> SB2
- J5 pad 2: Net-(U18-GNDA) -> SA2
- R1 pad 1: BRAKE -> +24V
- R1 pad 2: GND -> RESET
- R11 pad 1: BRAKE1 -> Net-(IC2-VDSTH)
- R11 pad 2: GND -> GNDPWR
- R12 pad 1: PWM1 -> Net-(State1.2-K)
- R12 pad 2: GND -> Net-(IC2-FF2)
- R13 pad 1: DIRECTION1 -> Net-(State1.1-K)
- R13 pad 2: GND -> Net-(IC2-FF1)
- R14 pad 1: Net-(D6-A) -> +24V
- R14 pad 2: Net-(D6-K) -> RESET
- R15 pad 1: Net-(D7-A) -> Net-(IC2-RDEAD)
- R15 pad 2: Net-(D7-K) -> GNDPWR
- R16 pad 1: Net-(D8-A) -> Net-(D6-A)
- R16 pad 2: Net-(D8-K) -> LED1
- R17 pad 1: Net-(D9-A) -> Net-(D7-A)
- R17 pad 2: Net-(D9-K) -> LED2
- R18 pad 1: Net-(U12-VOA) -> GHA0
- R19 pad 1: Net-(U12-VOB) -> GLA0
- R2 pad 1: PWM -> Net-(State2.1-K)
- R2 pad 2: GND -> Net-(IC3-FF1)
- R20 pad 2: Net-(U12-GNDA) -> SA1
- R22 pad 2: Net-(U17-GNDA) -> SB1
- R24 pad 1: Net-(U17-VOA) -> GHB0
- R25 pad 1: Net-(U17-VOB) -> GLB0
- R26 pad 1: Net-(U18-VOA) -> GHA
- R27 pad 1: Net-(U18-VOB) -> GLA
- R28 pad 2: Net-(U18-GNDA) -> SA2
- R3 pad 1: DIRECTION -> Net-(State2.2-K)
- R3 pad 2: GND -> Net-(IC3-FF2)
- R30 pad 2: Net-(U23-GNDA) -> SB2
- R32 pad 1: Net-(U23-VOA) -> GHB
- R33 pad 1: Net-(U23-VOB) -> GLB
- R4 pad 1: Net-(D2-A) -> Net-(IC3-RDEAD)
- R4 pad 2: Net-(D2-K) -> GNDPWR
- R5 pad 1: Net-(D3-A) -> +5V
- R5 pad 2: Net-(D3-K) -> Net-(IC3-VDSTH)
- R6 pad 1: Net-(D4-A) -> Net-(IC3-VDSTH)
- R6 pad 2: Net-(D4-K) -> GNDPWR
- R7 pad 1: Net-(D5-A) -> +5VA
- R7 pad 2: Net-(D5-K) -> Net-(IC2-VDSTH)
- U13 pad 3: Net-(U12-GNDA) -> SA1
- U14 pad 2: Net-(U12-GNDA) -> SA1
- U15 pad 2: Net-(U17-GNDA) -> SB1
- U16 pad 3: Net-(U17-GNDA) -> SB1
- U19 pad 3: Net-(U18-GNDA) -> SA2
- U20 pad 2: Net-(U18-GNDA) -> SA2
- U21 pad 2: Net-(U23-GNDA) -> SB2
- U22 pad 3: Net-(U23-GNDA) -> SB2
- U3 pad 1: PWM -> +3.3V
- U3 pad 10: Net-(D5-K) -> unconnected-(U3-VE2-Pad10)
- U3 pad 11: H1 -> PWMH1
- U3 pad 12: Net-(D4-K) -> PWML1
- U3 pad 13: Net-(D4-K) -> SR1
- U3 pad 14: +3.3V -> PHASE1
- U3 pad 2: DIRECTION -> GND
- U3 pad 3: Net-(D4-A) -> OPHASE1
- U3 pad 4: Net-(D4-A) -> OSR1
- U3 pad 5: Net-(U3-Pad5) -> OPWML1
- U3 pad 6: Net-(D5-A) -> OPWMH1
- U3 pad 7: GND -> unconnected-(U3-NIC-Pad7)
- U3 pad 8: L1 -> GND
- U3 pad 9: Net-(D5-K) -> GNDPWR
- U5 pad 1: PWM -> +3.3V
- U5 pad 10: Net-(D3-K) -> unconnected-(U5-VE2-Pad10)
- U5 pad 11: H2 -> PWMH2
- U5 pad 12: Net-(D2-K) -> PWML2
- U5 pad 13: Net-(D2-K) -> SR2
- U5 pad 14: +3.3V -> PHASE2
- U5 pad 2: Net-(U5-Pad2) -> GND
- U5 pad 3: Net-(D2-A) -> OPHASE2
- U5 pad 4: Net-(D2-A) -> OSR2
- U5 pad 5: Net-(U3-Pad5) -> OPWML2
- U5 pad 6: Net-(D3-A) -> OPWMH2
- U5 pad 7: GND -> unconnected-(U5-NIC-Pad7)
- U5 pad 8: L2 -> GND
- U5 pad 9: Net-(D3-K) -> GNDPWR
- U7 pad 10: unconnected-(U7-IO34-Pad10) -> OPWMH2
- U7 pad 11: BRAKE1 -> OPWML2
- U7 pad 12: unconnected-(U7-IO32-Pad12) -> OSR2
- U7 pad 13: DISABLE -> OPHASE2
- U7 pad 14: PWM1 -> OPWMH1
- U7 pad 15: unconnected-(U7-IO26-Pad15) -> OPWML1
- U7 pad 16: DIRECTION1 -> OSR1
- U7 pad 17: unconnected-(U7-IO14-Pad17) -> OPHASE1
- U7 pad 20: PWM -> LED1
- U7 pad 21: BRAKE -> LED2
- U7 pad 24: DIRECTION -> LED3
- U7 pad 34: CS -> unconnected-(U7-IO5-Pad34)
- U7 pad 35: CLK -> unconnected-(U7-IO18-Pad35)
- U7 pad 36: MOSI -> unconnected-(U7-IO23-Pad36)
- U7 pad 38: MISO -> unconnected-(U7-IO19-Pad38)
Routing:
- net +3.3V: track 245.3 -> 140.9 mm, vias 15 -> 6
- net GND: track 97.0 -> 7.30 mm, vias 46 -> 3
- net +12V: track 80.5 -> 0.00 mm
- net DISABLE: track 70.2 -> 0.00 mm, vias 2 -> 0
- net RESET: track 0.00 -> 54.6 mm, vias 0 -> 4
- net DIRECTION1: track 53.1 -> 0.00 mm, vias 2 -> 0
- net PWM: track 50.2 -> 0.00 mm, vias 3 -> 0
- net PWM1: track 46.1 -> 0.00 mm, vias 4 -> 0
- net DIRECTION: track 42.2 -> 0.00 mm, vias 4 -> 0
- net +5V: track 0.00 -> 40.7 mm, vias 0 -> 3
- net +5VA: track 0.00 -> 29.5 mm, vias 0 -> 4
- net +24V: track 6.51 -> 35.7 mm, vias 0 -> 3
- net Net-(U10-Pad5): track 23.4 -> 0.00 mm, vias 3 -> 0
- net BRAKE: track 21.8 -> 0.00 mm
- net Net-(U3-Pad5): track 20.4 -> 0.00 mm, vias 2 -> 0
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- added copper zone on B.Cu, net GND
- added copper zone on F.Cu, net GND
- added copper zone on F.Cu, net SA1
- added copper zone on F.Cu, net SA2
- added copper zone on F.Cu, net SB1
- added copper zone on F.Cu, net SB2
- removed copper zone on In1.Cu, net GND
- removed copper zone on F.Cu, net Net-(U12-GNDA)
- removed copper zone on F.Cu, net Net-(U17-GNDA)
- removed copper zone on F.Cu, net Net-(U18-GNDA)
- removed copper zone on F.Cu, net Net-(U23-GNDA)
