File: HTMDv2.1.kicad_sch (KiCad schematic)
At the start: 118 parts, among them IC1 TJA1441AT_0Z, J1 Conn_02x20_Odd_Even, J2 Conn_02x20_Odd_Even, J3 MothreCANConn, J4 XT60PW-F, J5 XT60PW-F, J6 Conn_01x06, SW1 SW_Push, SW2 SW_Push, U1 ADP3338AKCZ-3.3, U10 TC74LCXC00FT, U11 TC7S14FU, U12 ADuM7223, U13 SQJ180EP-T1_GE3, U14 SQJ180EP-T1_GE3, U15 SQJ180EP-T1_GE3, U16 SQJ180EP-T1_GE3, U17 ADuM7223, U18 ADuM7223, U19 SQJ180EP-T1_GE3, U2 NJM78L12SU3, U20 SQJ180EP-T1_GE3, U21 SQJ180EP-T1_GE3, U22 SQJ180EP-T1_GE3, U23 ADuM7223, U3 TC74LCXC00FT, U4 TC7S32FU, U5 TC74LCXC00FT, U6 TC7S14FU, U7 ESP32-PICO-D4, U8 TC74LCXC00FT, U9 TC7S32FU

Commit message: Artwork finish
Parts:
- removed C28, C33, C34, C39, C5: 0.1u, Capacitor_SMD:C_0402_1005Metric, symbol Device:C
- removed C29, C30, C31, C32, C35, C36, C37, C38, C6: 10u, Capacitor_SMD:C_0805_2012Metric, symbol Device:C
- removed C4: 1u, Capacitor_SMD:C_0402_1005Metric, symbol Device:C
- removed D10, D11, D12, D13: SS2040FL, 0-Myparts:SS2040FL, symbol Device:D
- removed D2, D3, D4, D5, D6, D7, D8, D9: BAT43XV2, 0-Myparts:BAT43XV2, symbol Device:D
- removed U10, U3, U5, U8: TC74LCXC00FT, 0-Myparts:TC74AC00FTEL, symbol 0-Myparts:TC74VHC00F
- removed U11, U6: TC7S14FU, 0-Myparts:TC7S14FU, symbol 0-Myparts:TC7S14FU
- removed U12, U17, U18, U23: ADuM7223, 0-Myparts:ADuM7223, symbol 0-Myparts:ADuM7223
- removed U2: NJM78L12SU3, 0-Myparts:REG_MCP1700T-3602E_MB, symbol 0-Myparts:NJM78L12SU3
- removed U4, U9: TC7S32FU, 0-Myparts:TC7S32FU, symbol 0-Myparts:TC7S32FU
- added D6, D7, D8, State1.1, State1.2, State2.1, State2.2: LED, LED_SMD:LED_0603_1608Metric_Pad1.05x0.95mm_HandSolder, symbol Device:LED
- added IC2, IC3: A3921KLPTR-T, 0-Myparts:A3944KLPTRT, symbol 0-Myparts:A3921KLPTR-T
- added R34: R, Resistor_SMD:R_0603_1608Metric_Pad0.98x0.95mm_HandSolder, symbol Device:R
- added SW3: SW_Push, 0-Myparts:SKRPABE010, symbol Switch:SW_Push
- added U3, U5: ADUM140E0BRWZ-RL, 0-Myparts:ADuM140ER, symbol 0-Myparts:ADUM140E0BRWZ-RL
- C10, C12, C23, C25: value 220p -> 0.1u; footprint Capacitor_SMD:C_0402_1005Metric -> Capacitor_SMD:C_0402_1005Metric_Pad0.74x0.62mm_HandSolder
- C11, C13, C24, C26: value 220p -> 10u; footprint Capacitor_SMD:C_0402_1005Metric -> Capacitor_SMD:C_0805_2012Metric_Pad1.18x1.45mm_HandSolder
- C14, C21, C22, C7, C8, C9: value 0.1u -> 10u; footprint Capacitor_SMD:C_0402_1005Metric -> Capacitor_SMD:C_0805_2012Metric_Pad1.18x1.45mm_HandSolder
- C20, C27: footprint Capacitor_SMD:C_0402_1005Metric -> Capacitor_SMD:C_0402_1005Metric_Pad0.74x0.62mm_HandSolder
- R1, R12, R13, R2, R3: footprint Resistor_SMD:R_0603_1608Metric -> Resistor_SMD:R_0603_1608Metric_Pad0.98x0.95mm_HandSolder
- R11: value 20k -> 1k; footprint Resistor_SMD:R_0603_1608Metric -> Resistor_SMD:R_0603_1608Metric_Pad0.98x0.95mm_HandSolder
- R14, R15, R4: value 1.8k -> 20k; footprint Resistor_SMD:R_0603_1608Metric -> Resistor_SMD:R_0603_1608Metric_Pad0.98x0.95mm_HandSolder
- R16, R17: value 1.8k -> R; footprint Resistor_SMD:R_0603_1608Metric -> Resistor_SMD:R_0603_1608Metric_Pad0.98x0.95mm_HandSolder
- R5, R7: value 1.8k -> 10k; footprint Resistor_SMD:R_0603_1608Metric -> Resistor_SMD:R_0603_1608Metric_Pad0.98x0.95mm_HandSolder
- R6: value 1.8k -> 1k; footprint Resistor_SMD:R_0603_1608Metric -> Resistor_SMD:R_0603_1608Metric_Pad0.98x0.95mm_HandSolder
Connections:
- net +24V: now also C12.1, C23.1, R1.1, R14.1, IC2.13 (VBB), IC3.13 (VBB)
- net +3.3V: now also U3.1 (VDD1), U5.1 (VDD1); no longer C14.1, C20.1, C21.1, C22.1, C27.1, C7.1, C8.1, C9.1
- net +5V: now also C10.1, C11.1, R5.1, IC3.20 (V5), State2.1.2 (A), State2.2.2 (A), U5.16 (VDD2)
- net GND: now also D6.1 (K), D7.1 (K), D8.1 (K), U3.2 (GND1), U3.8 (GND1), U5.2 (GND1), U5.8 (GND1); no longer C10.1, C11.1, C12.1, C13.1, C14.2, C20.2, C21.2, C22.2, C23.1, C24.1, C25.1, C26.1, C27.2, C7.2, C8.2, C9.2, R1.2, R11.2, R12.2, R13.2, R2.2, R3.2
- net GNDPWR: now also C10.2, C11.2, C12.2, C14.2, C20.2, C23.2, C24.2, C25.2, C26.2, C27.2, R11.2, R15.2, R4.2, R6.2, IC2.1 (VDRAIN), IC2.17 (GND), IC2.2 (LSS), IC2.29 (EP), IC3.1 (VDRAIN), IC3.17 (GND), IC3.2 (LSS), IC3.29 (EP), SW3.1, U3.15 (GND2), U3.9 (GND2), U5.15 (GND2), U5.9 (GND2)
- net at R4.1: now also IC3.27 (RDEAD)
- net SB1: now reaches J4.1, R22.2, U15.2, U16.3
- net SB1: now also C22.1, IC2.4 (SB)
- net GHB0: now reaches R24.1
- net GHB0: now also IC2.5 (GHB)
- net GLB0: now reaches R25.1
- net GLB0: now also IC2.3 (GLB)
- net SB2: now reaches J5.1, R30.2, U21.2, U22.3
- net SB2: now also C7.1, IC3.4 (SB)
- net OPWMH2: now reaches U7.10 (IO34)
- net OPWMH2: now also U5.6 (VID)
- net OSR2: now reaches U7.12 (IO32)
- net OSR2: now also U5.4 (VIB)
- net OPWML1: now reaches U7.15 (IO26)
- net OPWML1: now also U3.5 (VIC)
- net OPHASE1: now reaches U7.17 (IO14)
- net OPHASE1: now also U3.3 (VIA)
- net GLA: now reaches R27.1
- net GLA: now also IC3.12 (GLA)
- net SA1: now reaches J4.2, R20.2, U13.3, U14.2
- net SA1: now also C21.1, IC2.9 (CA)
- net at R16.1: now also D6.2 (A)
- net LED1: now reaches R16.2
- net LED1: now also U7.20 (IO13); no longer C25.2
- net RESET: now reaches R14.2
- net RESET: now also R1.2, IC2.24 (RESET), IC3.24 (RESET), SW3.2; no longer C23.2
- net SA2: now reaches J5.2, R28.2, U19.3, U20.2
- net SA2: now also C8.1, IC3.9 (CA)
- net at R6.1: now also R5.2, IC3.28 (VDSTH)
- net +5VA: now reaches R7.1
- net +5VA: now also C14.1, C20.1, IC2.20 (V5), State1.1.2 (A), State1.2.2 (A), U3.16 (VDD2)
- net at R7.2: now also R11.1, IC2.28 (VDSTH); no longer C13.2
- net GHA0: now reaches R18.1
- net GHA0: now also IC2.10 (GHA)
- net GLA0: now reaches R19.1
- net GLA0: now also IC2.12 (GLA)
- net LED2: now reaches R17.2
- net LED2: now also U7.21 (IO15); no longer C26.2
- net GHB: now reaches R32.1
- net GHB: now also IC3.5 (GHB)
- net GLB: now reaches R33.1
- net GLB: now also IC3.3 (GLB)
- net GHA: now reaches R26.1
- net GHA: now also IC3.10 (GHA)
- net at R15.1: now also IC2.27 (RDEAD)
- net at R17.1: now also D7.2 (A)
- removed net BRAKE: R1.1, U7.21 (IO15)
- net BRAKE1 renamed OPWML2
- net OPWML2: now also U5.5 (VIC); no longer R11.1
- net CLK: no longer names the net of U7.35 (IO18)
- net CS: no longer names the net of U7.34 (IO5)
- net DIRECTION: no longer names the net of R3.1
- net DIRECTION: now also State2.2.1 (K); no longer U7.24 (IO4)
- net DIRECTION1: no longer names the net of R13.1
- net DIRECTION1: now also State1.1.1 (K); no longer U7.16 (IO27)
- net DISABLE renamed OPHASE2
- net OPHASE2: now also U5.3 (VIA)
- net MISO: no longer names the net of U7.38 (IO19)
- net MOSI: no longer names the net of U7.36 (IO23)
- net PWM: no longer names the net of R2.1
- net PWM: now also State2.1.1 (K); no longer U7.20 (IO13)
- net PWM1: no longer names the net of R12.1
- net PWM1: now also State1.2.1 (K); no longer U7.14 (IO25)
- new net: C26.1, C27.1, IC2.8 (VREG)
- new net: C7.2, IC3.6 (CB)
- new net: IC2.25 (FF1), R13.2
- new net: C9.1, IC3.16 (CP1)
- new net: C24.1, C25.1, IC3.8 (VREG)
- new net: D8.2 (A), R34.1
- new net: C8.2, IC3.11 (SA)
- new net: IC3.25 (FF1), R2.2
- new net: IC3.26 (FF2), R3.2
- new net: C22.2, IC2.6 (CB)
- new net: C21.2, IC2.11 (SA)
- new net: C13.1, IC2.16 (CP1)
- new net: IC2.26 (FF2), R12.2
- new net CP1: C13.2, IC2.15 (CP2)
- new net CP2: C9.2, IC3.15 (CP2)
- new net LED3: R34.2, U7.24 (IO4)
- new net OPWMH1: U3.6 (VID), U7.14 (IO25)
- new net OSR1: U3.4 (VIB), U7.16 (IO27)
- new net PHASE1: IC2.19 (PHASE), U3.14 (VOA)
- new net PHASE2: IC3.19 (PHASE), U5.14 (VOA)
- new net PWMH1: IC2.23 (PWMH), U3.11 (VOD)
- new net PWMH2: IC3.23 (PWMH), U5.11 (VOD)
- new net PWML1: IC2.22 (PWML), U3.12 (VOC)
- new net PWML2: IC3.22 (PWML), U5.12 (VOC)
- new net SR1: IC2.21 (SR), U3.13 (VOB)
- new net SR2: IC3.21 (SR), U5.13 (VOB)
- no-connect marks 22 -> 29
Other:
- note removed: "デッドタイム≒400ns"
- note removed: "ロジック"
- moved on the sheet: C15, C16, C17, C18, C19, IC1, J4, J5, JP1, R10, R18, R19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
